File: pcb/host_board/control.sch (KiCad schematic (older format))
At the start: 50 parts, among them P301 USB_OTG, P302 CONN_01X04, P303 CONN_01X06, P304 CONN_01X06, P305 CONN_01X06, P306 CONN_01X06, P307 CONN_01X08, SW301 SW_PUSH, U301 STM32F072CBU, U302 TCA9548AR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

Commit message: added pdb schematic
Parts:
- P301: symbol USB_OTG -> USB_OTG-RESCUE-host_board
Changed lines of the file:
@@
 EESchema Schematic File Version 2
+LIBS:host_board-rescue
 LIBS:power
 LIBS:device
@@
 $Descr A4 11693 8268
 encoding utf-8
-Sheet 3 4
+Sheet 4 4
 Title ""
 Date ""
@@
 $EndComp
 $Comp
-L USB_OTG P301
+L USB_OTG-RESCUE-host_board P301
 U 1 1 56B6EFE2
 P 900 1700
+AR Path="/56B6EFE2" Ref="P301"  Part="1"
+AR Path="/56B5763E/56B6EFE2" Ref="P301"  Part="1"
 F 0 "P301" H 1225 1575 50  0000 C CNN
 F 1 "USB_OTG" H 900 1900 50  0000 C CNN
